File: diagrams/Bridge.kicad_sch (KiCad schematic)
At the start: 7 parts, among them J1 USB_A, J2 USB_A, J3 USB_A, J4 USB_A, J5 USB_A, U1 WeMos_D1_mini, U2 TSR1-2433E

Commit message: Added drawio diagrams and circuits
Connections:
- net at U1.1 (~{RST}): now also U1.3 (D0)
Changed lines of the file:
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@@
+	(wire
+		(pts
+			(xy 87.63 97.79) (xy 105.41 97.79)
+		)
+		(stroke
+			(width 0)
+			(type default)
+			(color 255 153 0 1)
+		)
+	)
 	(wire
 		(pts
@@
 	(wire
 		(pts
+			(xy 139.7 74.93) (xy 116.84 74.93)
+		)
+		(stroke
+			(width 0)
+			(type default)
+		)
+	)
+	(wire
+		(pts
 			(xy 171.45 152.4) (xy 182.88 152.4)
 		)
@@
 	(wire
 		(pts
+			(xy 87.63 100.33) (xy 105.41 100.33)
+		)
+		(stroke
+			(width 0)
+			(type default)
+		)
+	)
+	(wire
+		(pts
 			(xy 146.05 63.5) (xy 148.59 60.96)
 		)
@@
 	(wire
 		(pts
-			(xy 87.63 97.79) (xy 105.41 97.79)
-		)
-		(stroke
-			(width 0)
-			(type default)
-			(color 255 153 0 1)
-		)
-	)
-	(wire
-		(pts
 			(xy 93.98 107.95) (xy 93.98 85.09)
 		)
@@
 	(wire
 		(pts
+			(xy 115.57 85.09) (xy 116.84 86.36)
+		)
+		(stroke
+			(width 0)
+			(type default)
+		)
+	)
+	(wire
+		(pts
 			(xy 157.48 111.76) (xy 163.83 111.76)
 		)
@@
 	(wire
 		(pts
+			(xy 116.84 74.93) (xy 115.57 76.2)
+		)
+		(stroke
+			(width 0)
+			(type default)
+		)
+	)
+	(wire
+		(pts
 			(xy 185.42 97.79) (xy 185.42 74.93)
 		)
@@
 	(wire
 		(pts
+			(xy 138.43 86.36) (xy 139.7 86.36)
+		)
+		(stroke
+			(width 0)
+			(type default)
+		)
+	)
+	(wire
+		(pts
 			(xy 151.13 87.63) (xy 151.13 91.44)
 		)
@@
 	(wire
 		(pts
+			(xy 140.97 76.2) (xy 139.7 74.93)
+		)
+		(stroke
+			(width 0)
+			(type default)
+		)
+	)
+	(wire
+		(pts
 			(xy 128.27 116.84) (xy 128.27 118.11)
 		)
@@
 	(wire
 		(pts
+			(xy 140.97 85.09) (xy 140.97 76.2)
+		)
+		(stroke
+			(width 0)
+			(type default)
+		)
+	)
+	(wire
+		(pts
 			(xy 149.86 63.5) (xy 163.83 63.5)
 		)
@@
 	(wire
 		(pts
+			(xy 116.84 86.36) (xy 118.11 86.36)
+		)
+		(stroke
+			(width 0)
+			(type default)
+		)
+	)
+	(wire
+		(pts
 			(xy 152.4 109.22) (xy 157.48 114.3)
 		)
@@
 	(wire
 		(pts
-			(xy 87.63 100.33) (xy 105.41 100.33)
-		)
-		(stroke
-			(width 0)
-			(type default)
-		)
-	)
-	(wire
-		(pts
 			(xy 87.63 92.71) (xy 87.63 73.66)
 		)
@@
 	(wire
 		(pts
+			(xy 115.57 76.2) (xy 115.57 85.09)
+		)
+		(stroke
+			(width 0)
+			(type default)
+		)
+	)
+	(wire
+		(pts
 			(xy 172.72 97.79) (xy 185.42 97.79)
 		)
@@
 		)
 	)
+	(wire
+		(pts
+			(xy 139.7 86.36) (xy 140.97 85.09)
+		)
+		(stroke
+			(width 0)
+			(type default)
+		)
+	)
